Commit message: replace with new project: add imu_driver, nav2/slam configs, mapping/navigation launch

File: urdf/ylhb_chassis.urdf.xacro (robot description, xacro)
@@ -2,7 +2,7 @@
 <robot xmlns:xacro="http://www.ros.org/wiki/xacro" name="ylhb_chassis">
   <!-- 按实际车量尺寸改 -->
-  <xacro:property name="wheel_radius" value="0.10"/>
+  <xacro:property name="wheel_radius" value="0.15"/>
   <xacro:property name="base_length"  value="0.60"/>
-  <xacro:property name="base_width"   value="0.53"/>
+  <xacro:property name="base_width"   value="0.50"/>
   <xacro:property name="base_height"  value="0.30"/>
   <!-- 里程计的 child frame：base_link 投影到地面 -->

Commit message: add SerialPort driver and zdt motor control

File: urdf/ylhb_chassis.urdf.xacro (robot description, xacro)
@@ -30,10 +30,10 @@
     <origin xyz="-0.28 0 0.107" rpy="0 0 0"/>
   </joint>
-  <!-- 雷达：yaw 按实际安装角度标定 -->
+  <!-- 雷达：扫描 0° 即车头正方向（物理安装时雷达 0° 角/壳体背面朝车头） -->
   <link name="laser_link"/>
   <joint name="base_to_laser" type="fixed">
     <parent link="base_link"/>
     <child link="laser_link"/>
-    <origin xyz="-0.09 0 0.18" rpy="0 0 -1.5707963"/>
+    <origin xyz="-0.09 0 0.18" rpy="0 0 0"/>
   </joint>
 </robot>
